File: kicad_rgb_module.kicad_sch (KiCad schematic)
At the start: 37 parts, among them J1 Conn_HackConnect, SW1 TS-1088-AR02016, U1 STM32G030F6P6, U2 NCP114ASN330T1G

Commit message: Add diode to nRESET, decide on board sides for GerberSockets
Parts:
- added D9: 1N4148WS, Diode_SMD:D_SOD-323, symbol Diode:1N4148WS
Connections:
- net nRESET: now also D9.2 (A); no longer GS4.1 (RESET), J1.5
- new net nRESET-SAFE: D9.1 (K), GS4.1 (RESET), J1.5
Other:
- moved on the sheet: GS1, GS2, GS3, GS4, GS5, GS6, GS7, GS8
