File: kicad_rgb_module.kicad_sch (KiCad schematic)
At the start: 40 parts, among them J1 Conn_HackConnect, SW1 TS-1088-AR02016, U1 STM32G030F6P6, U2 NCP114ASN330T1G

Commit message: Add final order DL-21-v0.1 gerbers (with BAT54S->BAS40-04 change, but only in BOM and CPL csvs, not kicad). Fix too small via pads, DNP C1, revert mounting hole soldermask back to normal.
Parts:
- C1: now not fitted
Changed lines of the file:
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@@
 		(in_bom yes)
 		(on_board yes)
-		(dnp no)
+		(dnp yes)
 		(property "Reference" "C1"
 			(at 153.67 52.0699 0)
