File: kicad_rgb_module.kicad_sch (KiCad schematic)
At the start: 38 parts, among them J1 Conn_HackConnect, SW1 TS-1088-AR02016, U1 STM32G030F6P6, U2 NCP114ASN330T1G

Commit message: Change some GerberSockets and components
Parts:
- removed GS7: TEST_1, GerberSockets:TEST_1, symbol GerberSockets:TEST_1
- removed GS8: TEST_2, GerberSockets:TEST_2, symbol GerberSockets:TEST_2
- added GS7: 3V3, GerberSockets:3V3, symbol GerberSockets:3V3
- added GS8: SERIAL, GerberSockets:SERIAL, symbol GerberSockets:SERIAL
- FB1: LCSC Part C85815 -> C1002
- R1: LCSC Part C14663 -> C22962
Connections:
- net +3V3: now also GS7.1 (3V3)
- net SERIAL: now reaches U1.7 (PA0)
- net SERIAL: now also GS8.1 (SERIAL)
- no-connect marks 9 -> 8
Changed lines of the file:
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@@
 	)
 	(no_connect
-		(at 78.74 113.03)
-	)
-	(no_connect
 		(at 127 105.41)
 	)
@@
 	(wire
 		(pts
+			(xy 77.47 113.03) (xy 78.74 113.03)
+		)
+		(stroke
+			(width 0)
+			(type default)
+		)
+	)
+	(wire
+		(pts
 			(xy 127 113.03) (xy 128.27 113.03)
 		)
@@
 	(wire
 		(pts
+			(xy 247.65 144.78) (xy 259.08 144.78)
+		)
+		(stroke
+			(width 0)
+			(type default)
+		)
+	)
+	(wire
+		(pts
 			(xy 107.95 38.1) (xy 107.95 49.53)
 		)
@@
 	(wire
 		(pts
+			(xy 243.84 133.35) (xy 259.08 133.35)
+		)
+		(stroke
+			(width 0)
+			(type default)
+		)
+	)
+	(wire
+		(pts
 			(xy 214.63 120.65) (xy 226.06 120.65)
 		)
@@
 		)
 	)
+	(label "SERIAL"
+		(at 77.47 113.03 180)
+		(effects
+			(font
+				(size 1.27 1.27)
+			)
+			(justify right bottom)
+		)
+	)
 	(label "SWDIO"
 		(at 45.72 162.56 0)
@@
 		)
 	)
+	(label "SERIAL"
+		(at 247.65 144.78 0)
+		(effects
+			(font
+				(size 1.27 1.27)
+			)
+			(justify left bottom)
+		)
+	)
 	(label "JD_PWR"
 		(at 214.63 120.65 0)
@@
 			)
 		)
-		(property "LCSC Part" "C85815"
+		(property "LCSC Part" "C1002"
 			(at 130.81 38.1 90)
 			(effects
@@
 			)
 		)
-		(property "LCSC Part" "C14663"
+		(property "LCSC Part" "C22962"
 			(at 156.21 38.1 90)
 			(effects
@@
 	)
 	(symbol
-		(lib_id "GerberSockets:TEST_1")
-		(at 259.08 133.35 0)
+		(lib_id "power:GND")
+		(at 58.42 62.23 0)
 		(unit 1)
 		(exclude_from_sim no)
-		(in_bom no)
+		(in_bom yes)
 		(on_board yes)
 		(dnp no)
 		(fields_autoplaced yes)
-		(property "Reference" "GS7"
-			(at 259.08 130.302 0)
-			(do_not_autoplace yes)
+		(property "Reference" "#PWR06"
+			(at 58.42 68.58 0)
 			(effects
 				(font
 					(size 1.27 1.27)
 				)
+				(hide yes)
 			)
 		)
-		(property "Value" "TEST_1"
-			(at 259.08 133.35 0)
+		(property "Value" "GND"
+			(at 58.42 67.31 0)
 			(effects
 				(font
 					(size 1.27 1.27)
 				)
-				(hide yes)
 			)
 		)
-		(property "Footprint" "GerberSockets:TEST_1"
-			(at 259.08 139.954 0)
+		(property "Footprint" ""
+			(at 58.42 62.23 0)
 			(effects
 				(font
@@
 		)
 		(property "Datasheet" ""
-			(at 259.08 133.35 0)
+			(at 58.42 62.23 0)
 			(effects
 				(font
@@
 			)
 		)
-		(property "Description" "ASCII GerberSocket for net TEST_1"
-			(at 259.08 142.494 0)
-			(do_not_autoplace yes)
+		(property "Description" "Power symbol creates a global label with name \"GND\" , ground"
+			(at 58.42 62.23 0)
 			(effects
 				(font
@@
 		)
 		(instances
-			(project ""
+			(project "kicad_rgb_module"
 				(path "/9a8e7fbc-34f9-4889-88fa-a265258a8f63"
-					(reference "GS7")
+					(reference "#PWR06")
 					(unit 1)
 				)
@@
 	)
 	(symbol
-		(lib_id "GerberSockets:TEST_2")
+		(lib_id "GerberSockets:SERIAL")
 		(at 259.08 144.78 0)
 		(unit 1)
@@
 			)
 		)
-		(property "Value" "TEST_2"
+		(property "Value" "SERIAL"
 			(at 259.08 144.78 0)
 			(effects
@@
 			)
 		)
-		(property "Footprint" "GerberSockets:TEST_2"
+		(property "Footprint" "GerberSockets:SERIAL"
 			(at 259.08 151.384 0)
 			(effects
@@
 			)
 		)
-		(property "Description" "ASCII GerberSocket for net TEST_2"
+		(property "Description" "ASCII GerberSocket for net SERIAL"
 			(at 259.08 153.924 0)
 			(do_not_autoplace yes)
@@
 	)
 	(symbol
-		(lib_id "power:GND")
-		(at 58.42 62.23 0)
-		(unit 1)
-		(exclude_from_sim no)
-		(in_bom yes)
-		(on_board yes)
-		(dnp no)
-		(fields_autoplaced yes)
-		(property "Reference" "#PWR06"
-			(at 58.42 68.58 0)
-			(effects
-				(font
-					(size 1.27 1.27)
-				)
-				(hide yes)
-			)
-		)
-		(property "Value" "GND"
-			(at 58.42 67.31 0)
-			(effects
-				(font
-					(size 1.27 1.27)
-				)
-			)
-		)
-		(property "Footprint" ""
-			(at 58.42 62.23 0)
-			(effects
-				(font
-					(size 1.27 1.27)
-				)
-				(hide yes)
-			)
-		)
-		(property "Datasheet" ""
-			(at 58.42 62.23 0)
-			(effects
-				(font
-					(size 1.27 1.27)
-				)
-				(hide yes)
-			)
-		)
-		(property "Description" "Power symbol creates a global label with name \"GND\" , ground"
-			(at 58.42 62.23 0)
-			(effects
-				(font
-					(size 1.27 1.27)
-				)
-				(hide yes)
-			)
-		)
-		(pin "1"
-		)
-		(instances
-			(project "kicad_rgb_module"
-				(path "/9a8e7fbc-34f9-4889-88fa-a265258a8f63"
-					(reference "#PWR06")
-					(unit 1)
-				)
-			)
-		)
-	)
-	(symbol
 		(lib_id "Jacdac:jacdac_hole_PWR_MH3")
 		(at 224.79 36.83 0)
@@
 	)
 	(symbol
+		(lib_id "GerberSockets:3V3")
+		(at 259.08 133.35 0)
+		(unit 1)
+		(exclude_from_sim no)
+		(in_bom no)
+		(on_board yes)
+		(dnp no)
+		(fields_autoplaced yes)
+		(property "Reference" "GS7"
+			(at 259.08 130.302 0)
+			(do_not_autoplace yes)
+			(effects
+				(font
+					(size 1.27 1.27)
+				)
+			)
+		)
+		(property "Value" "3V3"
+			(at 259.08 133.35 0)
+			(effects
+				(font
+					(size 1.27 1.27)
+				)
+				(hide yes)
+			)
+		)
+		(property "Footprint" "GerberSockets:3V3"
+			(at 259.08 139.954 0)
+			(effects
+				(font
+					(size 1.27 1.27)
+				)
+				(hide yes)
+			)
+		)
+		(property "Datasheet" ""
+			(at 259.08 133.35 0)
+			(effects
+				(font
+					(size 1.27 1.27)
+				)
+				(hide yes)
+			)
+		)
+		(property "Description" "ASCII GerberSocket for net 3V3"
+			(at 259.08 142.494 0)
+			(do_not_autoplace yes)
+			(effects
+				(font
+					(size 1.27 1.27)
+				)
+				(hide yes)
+			)
+		)
+		(pin "1"
+		)
+		(instances
+			(project ""
+				(path "/9a8e7fbc-34f9-4889-88fa-a265258a8f63"
+					(reference "GS7")
+					(unit 1)
+				)
+			)
+		)
+	)
+	(symbol
 		(lib_id "power:GND")
 		(at 107.95 62.23 0)
@@
 					(unit 1)
 				)
+			)
+		)
+	)
+	(symbol
+		(lib_id "power:+3V3")
+		(at 243.84 133.35 0)
+		(unit 1)
+		(exclude_from_sim no)
+		(in_bom yes)
+		(on_board yes)
+		(dnp no)
+		(fields_autoplaced yes)
+		(property "Reference" "#PWR023"
+			(at 243.84 137.16 0)
+			(effects
+				(font
+					(size 1.27 1.27)
+				)
+				(hide yes)
+			)
+		)
+		(property "Value" "+3V3"
+			(at 243.84 128.27 0)
+			(effects
+				(font
+					(size 1.27 1.27)
+				)
+			)
+		)
+		(property "Footprint" ""
+			(at 243.84 133.35 0)
+			(effects
+				(font
+					(size 1.27 1.27)
+				)
+				(hide yes)
+			)
+		)
+		(property "Datasheet" ""
+			(at 243.84 133.35 0)
+			(effects
+				(font
+					(size 1.27 1.27)
+				)
+				(hide yes)
+			)
+		)
+		(property "Description" "Power symbol creates a global label with name \"+3V3\""
+			(at 243.84 133.35 0)
+			(effects
+				(font
+					(size 1.27 1.27)
+				)
+				(hide yes)
+			)
+		)
+		(pin "1"
+		)
+		(instances
+			(project "kicad_rgb_module"
+				(path "/9a8e7fbc-34f9-4889-88fa-a265258a8f63"
+					(reference "#PWR023")
+					(unit 1)
+				)

Commit message: Add test points
Parts:
- added TP1, TP2: TestPoint, Jacdac_Application:TestPoint_Pad_D1.0mm, symbol Connector:TestPoint
Connections:
- net +3V3: now also TP1.1
- net SERIAL: now also TP2.1
Other:
- moved on the sheet: D9, GS1, GS2, GS3, GS4, GS5, GS6, GS7, GS8

Commit message: Change design to use neopixel-style LED instead of regular RGB LED
Parts:
- removed D8: NH-B2020RGBA-GF, Jacdac_Application:LED-ARRAY-SMD_4P-L2.1-W2.1-TL_NH-B2020RGBA, symbol Jacdac_Application:FM-B2020RGBA-HG
- removed R4, R5, R6: 30R, Resistor_SMD:R_0603_1608Metric, symbol Device:R_US
- added D10: WS2812B, LED_SMD:LED_Inolux_IN-PI554FCH_PLCC4_5.0x5.0mm_P3.2mm, symbol Jacdac_Application:NeoPixel_WS2812B
- added R7: 300R, Resistor_SMD:R_0603_1608Metric, symbol Device:R_US
Connections:
- net +3V3: now also D10.1 (VDD)
- net GND: now also D10.3 (VSS)
- net RGB_B: no longer names the net of U1.14 (PA7)
- net RGB_G: no longer names the net of U1.15 (PB0/PB1/PB2/PA8)
- net RGB_R renamed LED_DIN
- net LED_DIN: now also R7.1
- new net: D10.4 (DIN), R7.2
- no-connect marks 8 -> 11

Commit message: Fix pin order and footprint of neopixel-style LED
Parts:
- added C5: 1uF, Capacitor_SMD:C_0603_1608Metric, symbol Device:C
- D10: footprint LED_SMD:LED_Inolux_IN-PI554FCH_PLCC4_5.0x5.0mm_P3.2mm -> Solderbit_Gamepad:NeoPixel_WS2812B
Connections:
- net +3V3: now also D10.3 (VDD), C5.2; no longer D10.1 (VDD)
- net GND: now also D10.1 (VSS), C5.1; no longer D10.3 (VSS)
- net at D10.2 (DIN): now also R7.2
- net at D10.4 (DOUT): no longer R7.2
Other:
- moved on the sheet: D10, R7

Commit message: Change BAT54 to BAS40-04 to reduce capacitance on JD_DATA
Parts:
- removed D1: BAT54S, Jacdac_Components:SOT-23_L2.9-W1.3-P1.90-LS2.4-BR, symbol Jacdac_Components:BAT54SLT1G
- added D1: BAS40-04, Package_TO_SOT_SMD:SOT-23, symbol Jacdac_Components:BAS40-04
- C1: now not fitted
- C5: LCSC Part (none) -> C15849; Package (none) -> 0603
Connections:
- net +3V3: now also D1.2
- net GND: now also D1.1
- net JD_DATA_MCU: now also D1.3
Changed lines of the file:
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@@
 		)
 	)
-	(text_box "D1 clamps JD_DATA\nto protect MCU."
+	(text_box "D1 clamps JD_DATA\nto protect MCU. BAS40 has lower capacitance compared to BAT54S"
 		(exclude_from_sim no)
-		(at 160.02 22.86 0)
-		(size 17.78 8.89)
+		(at 154.94 17.78 0)
+		(size 21.59 13.97)
 		(margins 0.9525 0.9525 0.9525 0.9525)
 		(stroke
@@
 		)
 	)
-	(text_box "R1/C1 form low-pass EMC filter."
+	(text_box "R1/C1 form low-pass EMC filter. Not fitted due to high capacitance on JD_DATA"
 		(exclude_from_sim no)
 		(at 161.29 53.34 0)
-		(size 12.7 10.16)
+		(size 13.97 16.51)
 		(margins 0.9525 0.9525 0.9525 0.9525)
 		(stroke
@@
 	(text_box "R1 > 0.12W in case 5V is mis-wired to JD_DATA. 5% tolerance is OK."
 		(exclude_from_sim no)
-		(at 137.16 19.05 0)
+		(at 133.35 17.78 0)
 		(size 17.78 12.7)
 		(margins 0.9525 0.9525 0.9525 0.9525)
@@
 	(wire
 		(pts
-			(xy 181.61 49.53) (xy 181.61 48.26)
+			(xy 180.34 45.72) (xy 180.34 48.26)
 		)
 		(stroke
@@
 	(wire
 		(pts
-			(xy 181.61 25.4) (xy 181.61 27.94)
+			(xy 180.34 27.94) (xy 180.34 30.48)
 		)
 		(stroke
@@
 	(wire
 		(pts
-			(xy 160.02 38.1) (xy 176.53 38.1)
+			(xy 160.02 38.1) (xy 175.26 38.1)
 		)
 		(stroke
@@
 		(in_bom yes)
 		(on_board yes)
-		(dnp no)
+		(dnp yes)
 		(property "Reference" "C1"
 			(at 153.67 52.0699 0)
@@
 	(symbol
 		(lib_id "power:+3V3")
-		(at 181.61 25.4 0)
+		(at 180.34 27.94 0)
 		(unit 1)
 		(exclude_from_sim no)
@@
 		(fields_autoplaced yes)
 		(property "Reference" "#PWR01"
-			(at 181.61 29.21 0)
+			(at 180.34 31.75 0)
 			(effects
 				(font
@@
 		)
 		(property "Value" "+3V3"
-			(at 181.61 20.32 0)
+			(at 180.34 22.86 0)
 			(effects
 				(font
@@
 		)
 		(property "Footprint" ""
-			(at 181.61 25.4 0)
+			(at 180.34 27.94 0)
 			(effects
 				(font
@@
 		)
 		(property "Datasheet" ""
-			(at 181.61 25.4 0)
+			(at 180.34 27.94 0)
 			(effects
 				(font
@@
 		)
 		(property "Description" "Power symbol creates a global label with name \"+3V3\""
-			(at 181.61 25.4 0)
+			(at 180.34 27.94 0)
 			(effects
 				(font
@@
 	(symbol
 		(lib_id "power:GND")
-		(at 181.61 49.53 0)
+		(at 180.34 48.26 0)
 		(unit 1)
 		(exclude_from_sim no)
@@
 		(fields_autoplaced yes)
 		(property "Reference" "#PWR04"
-			(at 181.61 55.88 0)
+			(at 180.34 54.61 0)
 			(effects
 				(font
@@
 		)
 		(property "Value" "GND"
-			(at 181.61 54.61 0)
+			(at 180.34 53.34 0)
 			(effects
 				(font
@@
 		)
 		(property "Footprint" ""
-			(at 181.61 49.53 0)
+			(at 180.34 48.26 0)
 			(effects
 				(font
@@
 		)
 		(property "Datasheet" ""
-			(at 181.61 49.53 0)
+			(at 180.34 48.26 0)
 			(effects
 				(font
@@
 		)
 		(property "Description" "Power symbol creates a global label with name \"GND\" , ground"
-			(at 181.61 49.53 0)
+			(at 180.34 48.26 0)
 			(effects
 				(font
@@
 	)
 	(symbol
-		(lib_id "power:+3V3")
-		(at 128.27 153.67 0)
+		(lib_id "Jacdac_Components:BAS40-04")
+		(at 182.88 38.1 90)
 		(unit 1)
 		(exclude_from_sim no)
@@
 		(dnp no)
 		(fields_autoplaced yes)
-		(property "Reference" "#PWR016"
-			(at 128.27 157.48 0)
+		(property "Reference" "D1"
+			(at 182.88 36.8299 90)
 			(effects
 				(font
 					(size 1.27 1.27)
 				)
-				(hide yes)
+				(justify right)
 			)
 		)
-		(property "Value" "+3V3"
-			(at 128.27 148.59 0)
+		(property "Value" "BAS40-04"
+			(at 182.88 39.3699 90)
 			(effects
 				(font
 					(size 1.27 1.27)
 				)
+				(justify right)
 			)
 		)
-		(property "Footprint" ""
-			(at 128.27 153.67 0)
+		(property "Footprint" "Package_TO_SOT_SMD:SOT-23"
+			(at 175.26 44.45 0)
 			(effects
 				(font
 					(size 1.27 1.27)
 				)
+				(justify left)
 				(hide yes)
 			)
 		)
-		(property "Datasheet" ""
-			(at 128.27 153.67 0)
+		(property "Datasheet" "http://www.vishay.com/docs/85701/bas40v.pdf"
+			(at 180.34 41.148 0)
 			(effects
 				(font
@@
 			)
 		)
-		(property "Description" "Power symbol creates a global label with name \"+3V3\""
-			(at 128.27 153.67 0)
+		(property "Description" "40V 0.2A Dual Small Signal Schottky Diodes"
+			(at 182.88 38.1 0)
+			(effects
+				(font
+					(size 1.27 1.27)
+				)
+				(hide yes)
+			)
+		)
+		(property "LCSC Part" "C7502688"
+			(at 182.88 38.1 90)
 			(effects
 				(font
@@
 		(pin "1"
 		)
+		(pin "2"
+		)
+		(pin "3"
+		)
 		(instances
-			(project "vm_rgb_led_0.1"
+			(project ""
 				(path "/9a8e7fbc-34f9-4889-88fa-a265258a8f63"
-					(reference "#PWR016")
+					(reference "D1")
 					(unit 1)
 				)
@@
 	)
 	(symbol
-		(lib_id "Jacdac_Components:BAT54SLT1G")
-		(at 182.88 38.1 90)
+		(lib_id "power:+3V3")
+		(at 128.27 153.67 0)
 		(unit 1)
 		(exclude_from_sim no)
@@
 		(on_board yes)
 		(dnp no)
-		(property "Reference" "D1"
-			(at 185.674 36.83 90)
-			(effects
-				(font
-					(size 1.27 1.27)
-				)
-				(justify left)
-			)
-		)
-		(property "Value" "BAT54S"
-			(at 190.246 38.862 90)
+		(fields_autoplaced yes)
+		(property "Reference" "#PWR016"
+			(at 128.27 157.48 0)
 			(effects
 				(font
 					(size 1.27 1.27)
 				)
-				(justify left)
+				(hide yes)
 			)
 		)
-		(property "Footprint" "Jacdac_Components:SOT-23_L2.9-W1.3-P1.90-LS2.4-BR"
-			(at 194.31 38.1 0)
+		(property "Value" "+3V3"
+			(at 128.27 148.59 0)
 			(effects
 				(font
 					(size 1.27 1.27)
 				)
-				(hide yes)
 			)
 		)
-		(property "Datasheet" "https://lcsc.com/product-detail/Schottky-Barrier-Diodes-SBD_ON_BAT54SLT1G_BAT54SLT1G_C19726.html"
-			(at 196.85 38.1 0)
+		(property "Footprint" ""
+			(at 128.27 153.67 0)
 			(effects
 				(font
@@
 			)
 		)
-		(property "Description" ""
-			(at 182.88 38.1 0)
+		(property "Datasheet" ""
+			(at 128.27 153.67 0)
 			(effects
 				(font
@@
 			)
 		)
-		(property "LCSC Part" "C19726"
-			(at 199.39 38.1 0)
+		(property "Description" "Power symbol creates a global label with name \"+3V3\""
+			(at 128.27 153.67 0)
 			(effects
 				(font
@@
 			)
 		)
-		(pin "3"
-		)
-		(pin "2"
-		)
 		(pin "1"
 		)
 		(instances
-			(project ""
+			(project "vm_rgb_led_0.1"
 				(path "/9a8e7fbc-34f9-4889-88fa-a265258a8f63"
-					(reference "D1")
+					(reference "#PWR016")
 					(unit 1)
 				)
@@
 			(at 163.83 123.19 0)
 			(effects
+				(font
+					(size 1.27 1.27)
+				)
+				(hide yes)
+			)
+		)
+		(property "LCSC Part" "C15849"
+			(at 163.83 123.19 0)
+			(effects
+				(font
+					(size 1.27 1.27)
+				)
+				(hide yes)
+			)
+		)
+		(property "Package" "0603"
+			(at 163.83 123.19 0)
+			(effects

Commit message: Remove GerberSockets to simplify the template, replace QR code with placeholder
Parts:
- removed D9: 1N4148WS, Diode_SMD:D_SOD-323, symbol Diode:1N4148WS
- removed GS1: GND, GerberSockets:GND, symbol GerberSockets:GND
- removed GS2: JD_DATA, GerberSockets:JD_DATA, symbol GerberSockets:JD_DATA
- removed GS3: JD_PWR, GerberSockets:JD_PWR, symbol GerberSockets:JD_PWR
- removed GS4: RESET, GerberSockets:RESET, symbol GerberSockets:RESET
- removed GS5: SWCLK, GerberSockets:SWCLK, symbol GerberSockets:SWCLK
- removed GS6: SWDIO~^, GerberSockets:SWDIO~^, symbol GerberSockets:SWDIO~^
- removed GS7: 3V3, GerberSockets:3V3, symbol GerberSockets:3V3
- removed GS8: SERIAL, GerberSockets:SERIAL, symbol GerberSockets:SERIAL
- removed TP1, TP2: TestPoint, Jacdac_Application:TestPoint_Pad_D1.0mm, symbol Connector:TestPoint
Other:
- moved on the sheet: C5, D10, R7

Commit message: Add jobfile for export, remove unused libs, leftover nets and traces in schematic and PCB
Connections:
- net nRESET-SAFE is gone; now on net nRESET: J1.5
- net SERIAL: no longer names the net of U1.7 (PA0)
- no-connect marks 11 -> 12
Changed lines of the file:
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@@
 		(at 127 110.49)
 	)
+	(no_connect
+		(at 78.74 113.03)
+	)
 	(wire
 		(pts
@@
 		(pts
 			(xy 88.9 45.72) (xy 99.06 45.72)
-		)
-		(stroke
-			(width 0)
-			(type default)
-		)
-	)
-	(wire
-		(pts
-			(xy 77.47 113.03) (xy 78.74 113.03)
 		)
 		(stroke
@@
 		)
 	)
+	(label "nRESET"
+		(at 22.86 179.07 0)
+		(effects
+			(font
+				(size 1.27 1.27)
+			)
+			(justify left bottom)
+		)
+	)
 	(label "JD_PWR"
 		(at 224.79 49.53 90)
@@
 		)
 	)
-	(label "SERIAL"
-		(at 77.47 113.03 180)
-		(effects
-			(font
-				(size 1.27 1.27)
-			)
-			(justify right bottom)
-		)
-	)
 	(label "SWDIO"
 		(at 45.72 162.56 0)
@@
 		)
 	)
-	(label "nRESET-SAFE"
-		(at 22.86 179.07 0)
-		(effects
-			(font
-				(size 1.27 1.27)
-			)
-			(justify left bottom)
-		)
-	)
