File: kicad_rgb_module.kicad_pcb (KiCad board)
At the start: 2 copper layers, 25 x 25 mm, 42 parts, among them J1 Conn_HackConnect, SW1 TS-1088-AR02016, U1 STM32G030F6P6, U2 NCP114ASN330T1G

Commit message: Change design to use neopixel-style LED instead of regular RGB LED
Parts:
- removed D8: NH-B2020RGBA-GF, Jacdac_Application:LED-ARRAY-SMD_4P-L2.1-W2.1-TL_NH-B2020RGBA
- removed R4, R5, R6: 30R, Resistor_SMD:R_0603_1608Metric
- added D10: WS2812B, LED_SMD:LED_Inolux_IN-PI554FCH_PLCC4_5.0x5.0mm_P3.2mm, F.Cu at (85.5, 75.0)
- added R7: 300R, Resistor_SMD:R_0603_1608Metric, F.Cu at (95.2, 80.2)
- moved D9 5.16 mm to (81.7, 80.0), turned to -90 degrees
- moved TP1 2.75 mm to (82.0, 75.0)
Connections:
- U1 pad 13: /RGB_R -> /LED_DIN
- U1 pad 14: /RGB_B -> unconnected-(U1-PA7-Pad14)
- U1 pad 15: /RGB_G -> unconnected-(U1-PB0/PB1/PB2/PA8-Pad15)
Routing:
- net Net-(D10-DIN): track 0.00 -> 19.1 mm
- net Net-(D8-R): track 18.2 -> 0.00 mm
- net Net-(D8-B): track 16.1 -> 0.00 mm
- net Net-(D8-G): track 12.5 -> 0.00 mm
- net /RGB_R: track 9.44 -> 0.00 mm
- net /LED_DIN: track 0.00 -> 9.44 mm
- net /nRESET: track 14.1 -> 22.5 mm
- net GND: track 90.3 -> 96.9 mm
- net JD_PWR: track 48.3 -> 51.1 mm
- net /RGB_B: track 2.41 -> 0.00 mm
- net /nRESET-SAFE: track 12.2 -> 14.3 mm
- net /RGB_G: track 2.01 -> 0.00 mm
- net /nFLASH: track 12.3 -> 13.1 mm
- net +3V3: track 60.2 -> 59.5 mm

Commit message: Fix pin order and footprint of neopixel-style LED
Parts:
- added C5: 1uF, Capacitor_SMD:C_0603_1608Metric, F.Cu at (84.3, 79.2)
- moved TP2 10.5 mm to (89.0, 75.0)
- turned D10 to -90 degrees
- turned D6 to 0 degrees
Connections:
- D10 pad 1: +3V3 -> GND
- D10 pad 2: unconnected-(D10-DOUT-Pad2) -> Net-(D10-DIN)
- D10 pad 3: GND -> +3V3
- D10 pad 4: Net-(D10-DIN) -> unconnected-(D10-DOUT-Pad4)
Routing:
- net GND: track 96.9 -> 108.5 mm
- net /nRESET: track 22.5 -> 17.5 mm
- net +3V3: track 59.5 -> 62.4 mm
- net /SERIAL: track 15.6 -> 13.6 mm, vias 2 -> 3
- net Net-(D6-Pad1): track 5.81 -> 4.03 mm
- net JD_PWR: track 51.1 -> 51.7 mm
